File: NIMRS-21Pin-Decoder.kicad_pcb (KiCad board)
At the start: 4 copper layers, 30 x 15.5 mm, 75 parts, among them J1 21Pin Loco Socket, J2 U.FL, Q1 MMDT3904, Q2 MMDT3904, U1 ESP32-S3FN8, U2 MAX98357A, U4 DRV8213DSGR, U60 TPS63070, U70 TPS63070, X1 40Mhz

Commit message: PCB Checkpoint
Parts:
- moved R7 0.30 mm to (20.7, 14.9)
- moved C76 0.14 mm to (15.4, 7.25)
- moved R1 0.12 mm to (23.4, 14.7)
Connections:
- U1 pad 38: /AUX3 -> /AMP_SD_MODE
- U1 pad 40: /VMOTOR_PG -> /AUX3
- U1 pad 41: /AMP_SD_MODE -> /AMP_LRCLK
- U1 pad 44: /AMP_LRCLK -> /VMOTOR_PG
- U1 pad 6: /MOTOR_CURRENT -> /TRACK_RIGHT
- U1 pad 9: /TRACK_RIGHT -> /MOTOR_CURRENT
Routing:
- net /rear: track 0.53 -> 32.6 mm, vias 1 -> 3
- net /front: track 0.56 -> 31.1 mm, vias 1 -> 3
- net /aux1: track 0.75 -> 30.7 mm, vias 1 -> 4
- net /aux2: track 0.75 -> 28.9 mm, vias 1 -> 3
- net /AUX4: track 1.52 -> 27.6 mm
- net /ZBDTA/D+: track 0.54 -> 26.5 mm, vias 1 -> 2
- net /ZBCLK/D-: track 0.54 -> 26.2 mm, vias 1 -> 2
- net /AUX3: track 0.66 -> 24.2 mm, vias 1 -> 3
- net /+V_SENSE: track 1.62 -> 19.3 mm, vias 1 -> 2
- net /VMOTOR_PG: track 0.60 -> 14.5 mm, vias 1 -> 2
- net /AUX5: track 1.55 -> 15.2 mm
- net /AMP_LRCLK: track 0.00 -> 11.9 mm, vias 0 -> 2
- net /TRACK_LEFT: track 1.52 -> 13.2 mm, vias 1 -> 2
- net /TRACK_RIGHT: track 1.79 -> 12.4 mm, vias 1 -> 2
- net /FRONT: track 0.00 -> 8.70 mm, vias 0 -> 2
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
Commit message: PCB RC1
Parts:
- removed R2: 10kΩ, Resistor_SMD:R_0805_2012Metric_Pad1.20x1.40mm_HandSolder
- added H1: ~, PCM_JLCPCB:Hole_Tooling_JLCPCB, F.Cu at (1.00, 18.5)
- added H2: ~, PCM_JLCPCB:Hole_Tooling_JLCPCB, F.Cu at (29.0, 18.5)
- added H3: ~, PCM_JLCPCB:Hole_Tooling_JLCPCB, F.Cu at (29.0, -3.00)
- added H4: ~, PCM_JLCPCB:Hole_Tooling_JLCPCB, F.Cu at (1.00, -3.00)
- added PN1: ~, PCM_JLCPCB:Part_Num_JLCPCB, F.Cu at (15.0, 18.4)
- added REF**: MouseBites, Cosmetic, JLCPCB, 1.6mm, PCM_JLCPCB:MouseBites, Cosmetic, JLCPCB, 1.6mm, F.Cu at (0.50, 15.5)
- added REF**: MouseBites, Cosmetic, JLCPCB, 1.6mm, PCM_JLCPCB:MouseBites, Cosmetic, JLCPCB, 1.6mm, F.Cu at (6.50, 0.00)
- added REF**: MouseBites, Cosmetic, JLCPCB, 1.6mm, PCM_JLCPCB:MouseBites, Cosmetic, JLCPCB, 1.6mm, F.Cu at (23.5, 15.5)
- added REF**: MouseBites, Cosmetic, JLCPCB, 1.6mm, PCM_JLCPCB:MouseBites, Cosmetic, JLCPCB, 1.6mm, F.Cu at (29.5, 0.00)
- added TP1: Test Point, Custom_Footprints:TestPoint_Pad_D1.0mm, B.Cu at (26.2, 5.55)
- added TP2: Test Point, Custom_Footprints:TestPoint_Pad_D1.0mm, B.Cu at (8.95, 1.15)
- added TP3: Test Point, Custom_Footprints:TestPoint_Pad_D1.0mm, B.Cu at (13.4, 7.25)
- added TP4: Test Point, Custom_Footprints:TestPoint_Pad_D1.0mm, B.Cu at (24.4, 14.5)
- added TP5: Test Point, Custom_Footprints:TestPoint_Pad_D1.0mm, B.Cu at (26.2, 11.5)
- added TP6: Test Point, Custom_Footprints:TestPoint_Pad_D1.0mm, B.Cu at (6.55, 3.88)
- added TP7: Test Point, Custom_Footprints:TestPoint_Pad_D1.0mm, B.Cu at (26.9, 9.65)
- D1, D2, D3, D4: footprint PCM_JLCPCB:D_SOD-323 -> Custom_Footprints:D_SOD-323
- U4: footprint Package_SON:WSON-8-1EP_2x2mm_P0.5mm_EP0.9x1.6mm -> Custom_Footprints:WSON-8-1EP_2x2mm_P0.5mm_EP0.9x1.6mm
- moved R11 20.1 mm to (6.90, 14.5)
- moved R1 4.64 mm to (27.2, 12.2), turned to -90 degrees
- moved C11 0.49 mm to (20.4, 5.77)
- moved R73 0.29 mm to (18.5, 7.05), turned to 90 degrees
- moved C10 0.23 mm to (25.4, 14.8)
- moved C13 0.18 mm to (29.0, 3.95)
- moved X1 0.15 mm to (27.7, 14.2)
- moved R72 0.11 mm to (16.8, 7.75)
- moved L3 0.11 mm to (28.3, 11.9)
- moved L4 0.10 mm to (28.6, 5.30)
- moved C76 0.10 mm to (15.5, 7.25)
- moved R10 0.07 mm to (7.78, 9.65)
Connections:
- U1 pad 10: /+V_SENSE -> /MOTOR_CURRENT
- U1 pad 11: /INPUT2/AUX8 -> /+V_SENSE
- U1 pad 12: /INPUT1/AUX7 -> /INPUT2/AUX8
- U1 pad 13: unconnected-(U1-GPIO8-Pad13) -> /INPUT1/AUX7
- U1 pad 14: unconnected-(U1-GPIO9-Pad14) -> /AUX1
- U1 pad 15: unconnected-(U1-GPIO10-Pad15) -> /AUX2
- U1 pad 16: /MOTOR_GAIN_SEL -> /REAR
- U1 pad 18: /AUX2 -> /FRONT
- U1 pad 23: /MOTOR_2 -> unconnected-(U1-GPIO17-Pad23)
- U1 pad 39: /MOTOR_1 -> /MOTOR_GAIN_SEL
- U1 pad 45: /REAR -> /MOTOR_2
- U1 pad 47: /FRONT -> /MOTOR_1
- U1 pad 48: /AUX1 -> unconnected-(U1-MTMS-Pad48)
- U1 pad 9: /MOTOR_CURRENT -> unconnected-(U1-GPIO4-Pad9)
Routing:
- net +3V3: track 19.9 -> 45.4 mm, vias 14 -> 16
- net /MOTOR_1: track 1.63 -> 24.2 mm
- net /MOTOR_2: track 2.70 -> 25.1 mm
- net /3V3_PG/ESP_EN: track 1.45 -> 22.9 mm, vias 1 -> 3
- net /MOTOR_GAIN_SEL: track 4.52 -> 24.8 mm, vias 2 -> 4
- net /VMOTOR_PG: track 14.5 -> 28.2 mm, vias 2 -> 4
- net /AUX5: track 15.2 -> 25.3 mm, vias 2 -> 4
- net /Track_Right: track 45.9 -> 38.1 mm
- net /REAR: track 2.26 -> 7.50 mm
- net /ESP32_TX: track 0.00 -> 4.70 mm, vias 0 -> 2
- net Net-(U1-U0TXD): track 5.68 -> 1.16 mm, vias 2 -> 0
- net GND: track 55.4 -> 59.0 mm, vias 58 -> 60
- net /MOTOR_CURRENT: track 32.7 -> 36.0 mm
- net /AUX2: track 7.98 -> 5.91 mm
- net /ESP32_RX: track 0.78 -> 2.13 mm
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- added copper zone on F.Cu, net GND
Other:
- board size 30 x 15.5 mm -> 30 x 23.5 mm
- board text added: "3V3"
- board text added: "EN/3V3_PG"
- board text added: "GND"
- board text added: "IO0"
- board text added: "IO45"
- board text added: "RX"
- board text added: "R_IPROPI"
- board text added: "TX"

Commit message: Center PCB, Tidy up for r/PrintedCurcuitBoard
Parts:
- moved C1 165.6 mm to (161.6, 102.5)
- moved C10 165.6 mm to (159.4, 112.0)
- moved C11 165.6 mm to (154.4, 103.0)
- moved C12 165.6 mm to (163.1, 104.5)
- moved C13 165.6 mm to (163.0, 101.2)
- moved C15 165.6 mm to (151.1, 107.4)
- moved C16 165.6 mm to (150.6, 107.9)
- moved C17 165.6 mm to (142.3, 104.7)
- moved C2 165.6 mm to (159.5, 100.2)
- moved C4 165.6 mm to (157.7, 100.2)
- moved C5 165.6 mm to (163.2, 108.6)
- moved C6 165.6 mm to (152.3, 106.2)
- moved C60 165.6 mm to (144.7, 102.1)
- moved C61 165.6 mm to (144.7, 103.6)
- moved C62 165.6 mm to (146.7, 105.8)
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