File: NIMRS-21Pin-Decoder.kicad_sch (KiCad schematic)
At the start: 75 parts, among them J1 21Pin Loco Socket, J2 U.FL, Q1 MMDT3904, Q2 MMDT3904, U1 ESP32-S3FN8, U2 MAX98357A, U4 DRV8213DSGR, U60 TPS63070, U70 TPS63070, X1 40Mhz

Commit message: PCB Checkpoint
Connections:
- net AMP_LRCLK: now also U1.41 (GPIO36); no longer U1.44 (MTCK)
- net AMP_SD_MODE: now also U1.38 (GPIO33); no longer U1.41 (GPIO36)
- net AUX3: now also U1.40 (GPIO35); no longer U1.38 (GPIO33)
- net MOTOR_CURRENT: now also U1.9 (GPIO4); no longer U1.6 (GPIO1)
- net TRACK_RIGHT: now also U1.6 (GPIO1); no longer U1.9 (GPIO4)
- net VMOTOR_PG: now also U1.44 (MTCK); no longer U1.40 (GPIO35)
Changed lines of the file:
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@@
-		)
-	)
-	(label "AUX3"
-		(at 198.12 50.8 0)
-		(effects
-			(font
-				(size 1.27 1.27)
-			)
-			(justify left bottom)
 		)
 	)
@@
 		)
 	)
-	(label "AMP_LRCLK"
-		(at 198.12 66.04 0)
-		(effects
-			(font
-				(size 1.27 1.27)
-			)
-			(justify left bottom)
-		)
-	)
 	(label "INPUT1{slash}AUX7"
 		(at 78.74 30.48 180)
@@
 		)
 	)
-	(label "AMP_SD_MODE"
-		(at 198.12 58.42 0)
-		(effects
-			(font
-				(size 1.27 1.27)
-			)
-			(justify left bottom)
-		)
-	)
 	(label "Speaker+"
 		(at 266.7 134.62 0)
@@
 		)
 	)
+	(label "TRACK_LEFT"
+		(at 152.4 33.02 180)
+		(effects
+			(font
+				(size 1.27 1.27)
+			)
+			(justify right bottom)
+		)
+	)
 	(label "Motor2"
 		(at 109.22 40.64 0)
@@
 		)
 	)
+	(label "AMP_LRCLK"
+		(at 198.12 58.42 0)
+		(effects
+			(font
+				(size 1.27 1.27)
+			)
+			(justify left bottom)
+		)
+	)
 	(label "TRACK_LEFT"
 		(at 314.96 7.62 0)
@@
 		)
 	)
-	(label "VMOTOR_PG"
-		(at 198.12 55.88 0)
-		(effects
-			(font
-				(size 1.27 1.27)
-			)
-			(justify left bottom)
-		)
-	)
 	(label "FRONT"
 		(at 198.12 71.12 0)
@@
 		)
 	)
-	(label "TRACK_LEFT"
-		(at 152.4 33.02 180)
-		(effects
-			(font
-				(size 1.27 1.27)
-			)
-			(justify right bottom)
-		)
-	)
 	(label "AMP_DIN"
 		(at 241.3 134.62 180)
@@
 		)
 	)
-	(label "TRACK_RIGHT"
-		(at 152.4 38.1 180)
-		(effects
-			(font
-				(size 1.27 1.27)
-			)
-			(justify right bottom)
-		)
-	)
 	(label "+V_SENSE"
 		(at 335.28 7.62 0)
@@
 		)
 	)
+	(label "AUX3"
+		(at 198.12 55.88 0)
+		(effects
+			(font
+				(size 1.27 1.27)
+			)
+			(justify left bottom)
+		)
+	)
 	(label "AUX6"
 		(at 78.74 35.56 180)
@@
 		)
 	)
+	(label "TRACK_RIGHT"
+		(at 152.4 30.48 180)
+		(effects
+			(font
+				(size 1.27 1.27)
+			)
+			(justify right bottom)
+		)
+	)
 	(label "ZBDTA{slash}D+"
 		(at 78.74 43.18 180)
@@
 		)
 	)
+	(label "AMP_SD_MODE"
+		(at 198.12 50.8 0)
+		(effects
+			(font
+				(size 1.27 1.27)
+			)
+			(justify left bottom)
+		)
+	)
 	(label "Speaker-"
 		(at 78.74 53.34 180)
@@
 		)
 	)
+	(label "MOTOR_CURRENT"
+		(at 152.4 38.1 180)
+		(effects
+			(font
+				(size 1.27 1.27)
+			)
+			(justify right bottom)
+		)
+	)
 	(label "front"
 		(at 88.9 124.46 180)
@@
 		)
 	)
+	(label "VMOTOR_PG"
+		(at 198.12 66.04 0)
+		(effects
+			(font
+				(size 1.27 1.27)
+			)
+			(justify left bottom)
+		)
+	)
 	(label "ESP32_RX"
 		(at 205.74 78.74 0)
@@
 		)
 	)
-	(label "MOTOR_CURRENT"
-		(at 152.4 30.48 180)
-		(effects
-			(font
-				(size 1.27 1.27)
-			)
-			(justify right bottom)
-		)
-	)

Commit message: PCB RC1
Parts:
- removed R2: 10kΩ, Resistor_SMD:R_0805_2012Metric_Pad1.20x1.40mm_HandSolder, symbol Device:R
- added H1, H2, H3, H4: ~, PCM_JLCPCB:Hole_Tooling_JLCPCB, symbol PCM_JLCPCB-Manufacturing:Tooling Hole, PCM_JLCPCB, 1.152mm
- added PN1: ~, PCM_JLCPCB:Part_Num_JLCPCB, symbol PCM_JLCPCB-Manufacturing:Part Number, PCM_JLCPCB, 0.8x0.15mm
- added TP1, TP2, TP3, TP4, TP5, TP6, TP7: Test Point, Custom_Footprints:TestPoint_Pad_D1.0mm, symbol Connector:TestPoint
- D1, D2, D3, D4: footprint PCM_JLCPCB:D_SOD-323 -> Custom_Footprints:D_SOD-323
- R11: now left out of the parts list
- U2: LCSC (none) -> C910544
- U4: footprint Package_SON:WSON-8-1EP_2x2mm_P0.5mm_EP0.9x1.6mm -> Custom_Footprints:WSON-8-1EP_2x2mm_P0.5mm_EP0.9x1.6mm
Connections:
- net +3V3: now also TP2.1
- net +V_SENSE: now also U1.11 (GPIO6); no longer U1.10 (GPIO5)
- net 3V3_PG/ESP_EN: now also TP3.1
- net AUX1: now also U1.14 (GPIO9); no longer U1.48 (MTMS)
- net AUX2: now also U1.15 (GPIO10); no longer U1.18 (GPIO13)
- net ESP32_RX: now also TP5.1
- net ESP32_TX: now also TP4.1
- net FRONT: now also U1.18 (GPIO13); no longer U1.47 (MTDI)
- net GND: now also TP6.1
- net INPUT1/AUX7: now also U1.13 (GPIO8); no longer U1.12 (GPIO7)
- net INPUT2/AUX8: now also U1.12 (GPIO7); no longer U1.11 (GPIO6)
- net IO0: now also TP1.1
- net MOTOR_1: now also U1.47 (MTDI); no longer U1.39 (GPIO34)
- net MOTOR_2: now also U1.45 (MTDO); no longer U1.23 (GPIO17)
- net MOTOR_CURRENT: now also U1.10 (GPIO5); no longer U1.9 (GPIO4)
- net MOTOR_GAIN_SEL: now also U1.39 (GPIO34); no longer U1.16 (GPIO11)
- net REAR: now also U1.16 (GPIO11); no longer U1.45 (MTDO)
- net at U1.51 (GPIO45): now also TP7.1
Other:
- note added: "VMOTOR is 9V"
- company: (none) -> Kea Studios
- title: (none) -> NIMRS-21Pin-Decoder
- moved on the sheet: C1, C10, C11, C12, C13, C15, C16, C17, C2, C4, C5, C6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

Commit message: Center PCB, Tidy up for r/PrintedCurcuitBoard
Other:
- moved on the sheet: C60, C61, C62, C63, C64, C65, C66, C67, C70, C71, C72, C73
